File: GWifi/GWifi.sch (EAGLE design)
At the start: 29 parts, among them U1 TSR12450, X1 2.1MMJACKTHM, X2 5268-02, X3 5268-02, X4 5268-03

Commit message: gpio description, sch pdf added
Other:
- note added: "LED1: GPIO22 / OUTPUT"
- note added: "LED2: GPIO24 / OUTPUT"
- note added: "LED3: GPIO23 / OUTPUT"
- note added: "SW1: GPIO4 / INPUT"
- note added: "SW2: GPIO17 / INPUT"
- note added: "SW3: GPIO27 / INPUT"
Changed lines of the file:
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@@
 <sheet>
 <plain>
+<text x="198.12" y="68.58" size="1.778" layer="94">SW1: GPIO4 / INPUT</text>
+<text x="198.12" y="66.04" size="1.778" layer="94">SW2: GPIO17 / INPUT</text>
+<text x="198.12" y="63.5" size="1.778" layer="94">SW3: GPIO27 / INPUT</text>
+<text x="198.12" y="55.88" size="1.778" layer="94">LED1: GPIO22 / OUTPUT</text>
+<text x="198.12" y="53.34" size="1.778" layer="94">LED2: GPIO24 / OUTPUT</text>
+<text x="198.12" y="50.8" size="1.778" layer="94">LED3: GPIO23 / OUTPUT</text>
 </plain>
 <instances>
