File: GCharger/GCharger.sch (EAGLE design)
At the start: 0 parts

Commit message: Gcharger Board
Parts:
- added C1, C2, C4, C5: (no value), Gcharger:C0603(1608)
- added C3, C7: DNP, g-project:C0603(1608)
- added C6, C8: 0.1uF monolithic, adafruit:C-US050-024X044
- added H1, H2, H3, H4: MOUNT-PAD-ROUND3.2, OSSI:MOUNT-PAD-ROUND3.2
- added JP1, JP2: (no value), adafruit:PINHD-1X1CB
- added LED1, LED2: Red, SparkFun-LED:LED3MM
- added LED3: Green, SparkFun-LED:LED3MM
- added R1, R12, R14, R6: 47k, g-project:R-US_FLIPFLOP
- added R10, R16, R4: 1.5k, g-project:R-US_FLIPFLOP
- added R11, R5: 10k, 1%, g-project:R-US_FLIPFLOP
- added R13, R15, R3, R9: 4.7k, g-project:R-US_FLIPFLOP
- added R2, R7: 0.1, 1% Current Sense, SparkFun-Resistors:RESISTOR1206
- added R8: 510, g-project:R-US_FLIPFLOP
- added S1: (no value), WaterDrop:SWITCH
- added TVS1, TVS2: SD0, Gcharger:SD0
- added U1, U2: INA169, Gcharger:INA169
- added U3: TLV2462, Gcharger:TLV2462
- added U4: ARDUINOR3-TPLACE, Gcharger:ARDUINOR3-TPLACE
- added X1, X4, X7: 5268-02, OSSI:5268-02
- added X2, X5: USB-B, Gcharger:USB+SHIELD
- added X3, X6: USB-A-Recep, Gcharger:USB-787616
Connections:
- new net +5V: C1.2, C4.2, C8.1, R12.2, R14.2, U1.V+, U2.V+, U3.P$8, U4.5V
- new net +5V_USB_1: C2.2, R2.1, TVS1.P$1, U1.VIN+, X2.VBUS
- new net +5V_USB_2: C5.2, R7.1, TVS2.P$1, U2.VIN+, X5.VBUS
- new net CURRENT1: C3.1, JP1.1, R5.2, U1.OUT, U3.P$3
- new net CURRENT2: C7.1, JP2.1, R11.2, U2.OUT, U3.P$5
- new net GND: C1.1, C3.2, C4.1, C6.2, C7.2, C8.2, LED1.C, LED2.C, LED3.C, R1.2, R11.1, R5.1, R6.2, R8.2, S1.P$1, U1.GND, U2.GND, U3.P$4, U4.GND, U4.GND1, U4.GND2, X1.2, X4.2, X7.2
- new net I_ADC1: U3.P$1, U3.P$2, U4.A0
- new net I_ADC2: U3.P$6, U3.P$7, U4.A1
- new net I_GND1: C2.1, TVS1.P$2, X2.GND, X3.4GND
- new net I_GND2: C5.1, TVS2.P$2, X5.GND, X6.4GND
- new net LED1: R16.2, U4.D12
- new net N$1: X5.D-, X6.2D-
- new net N$10: LED2.A, R10.1
- new net N$11: LED1.A, R4.1
- new net N$12: LED3.A, R16.1
- new net N$13: R14.1, R15.1, X7.1
- new net N$2: X5.D+, X6.3D+
- new net N$3: R1.1, R3.2, X1.1
- new net N$4: X2.D-, X3.2D-
- new net N$5: X2.D+, X3.3D+
- new net N$6: R7.2, U2.VIN-, X6.1VBUS
- new net N$7: R12.1, R13.1, S1.P$2
- new net N$8: R6.1, R9.2, X4.1
- new net N$9: R2.2, U1.VIN-, X3.1VBUS
- new net OUT1: R3.1, R4.2, U4.D9
- new net OUT2: R10.2, R9.1, U4.D10
- new net STRUT_GND: C6.1, H1.MOUNT, R8.1, X2.S1, X2.S2, X3.S1, X3.S2, X5.S1, X5.S2, X6.S1, X6.S2
- new net SW1: R13.2, U4.D2
- new net SW2: R15.2, U4.D3
Other:
- note added: "Charger Side"
- note added: "Indicator LED"
- note added: "Input 1 (Option)"
- note added: "Phone Side"
- note added: "SSR Control 1"
- note added: "SSR Control 2 (Option)"
- note added: "Test Button"

Commit message: gerber file added
Parts:
- added H5: MOUNT-PAD-ROUND3.2, OSSI:MOUNT-PAD-ROUND3.2
- C1, C4: value (none) -> 0.1uF
- C2, C5: value (none) -> 0.01uF
Other:
- moved on the sheet: H3, H4
Changed lines of the file:
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@@
 <part name="X3" library="Gcharger" deviceset="USB-787616" device="" value="USB-A-Recep"/>
 <part name="X6" library="Gcharger" deviceset="USB-787616" device="" value="USB-A-Recep"/>
-<part name="H3" library="OSSI" deviceset="MOUNT-PAD-ROUND" device="3.2"/>
+<part name="H4" library="OSSI" deviceset="MOUNT-PAD-ROUND" device="3.2"/>
 <part name="H2" library="OSSI" deviceset="MOUNT-PAD-ROUND" device="3.2"/>
-<part name="H4" library="OSSI" deviceset="MOUNT-PAD-ROUND" device="3.2"/>
+<part name="H5" library="OSSI" deviceset="MOUNT-PAD-ROUND" device="3.2"/>
 <part name="U4" library="Gcharger" deviceset="ARDUINOR3" device="-TPLACE"/>
 <part name="C8" library="adafruit" deviceset="C-US" device="050-024X044" value="0.1uF monolithic"/>
@@
 <part name="TVS1" library="Gcharger" deviceset="SD0" device=""/>
 <part name="TVS2" library="Gcharger" deviceset="SD0" device=""/>
-<part name="C2" library="Gcharger" deviceset="C" device="0603(1608)"/>
-<part name="C5" library="Gcharger" deviceset="C" device="0603(1608)"/>
-<part name="C1" library="Gcharger" deviceset="C" device="0603(1608)"/>
-<part name="C4" library="Gcharger" deviceset="C" device="0603(1608)"/>
+<part name="C2" library="Gcharger" deviceset="C" device="0603(1608)" value="0.01uF"/>
+<part name="C5" library="Gcharger" deviceset="C" device="0603(1608)" value="0.01uF"/>
+<part name="C1" library="Gcharger" deviceset="C" device="0603(1608)" value="0.1uF"/>
+<part name="C4" library="Gcharger" deviceset="C" device="0603(1608)" value="0.1uF"/>
 <part name="P+6" library="supply1" deviceset="+5V" device=""/>
 <part name="P+7" library="supply1" deviceset="+5V" device=""/>
+<part name="H3" library="OSSI" deviceset="MOUNT-PAD-ROUND" device="3.2"/>
 </parts>
 <sheets>
@@
 <instance part="X3" gate="G$1" x="55.88" y="99.06"/>
 <instance part="X6" gate="G$1" x="137.16" y="99.06"/>
-<instance part="H3" gate="G$1" x="71.12" y="226.06"/>
+<instance part="H4" gate="G$1" x="71.12" y="226.06"/>
 <instance part="H2" gate="G$1" x="27.94" y="215.9"/>
-<instance part="H4" gate="G$1" x="71.12" y="215.9"/>
+<instance part="H5" gate="G$1" x="71.12" y="215.9"/>
 <instance part="U4" gate="G$1" x="233.68" y="132.08" rot="R90"/>
 <instance part="C8" gate="G$1" x="256.54" y="190.5"/>
@@
 <instance part="P+6" gate="1" x="20.32" y="60.96"/>
 <instance part="P+7" gate="1" x="101.6" y="60.96"/>
+<instance part="H3" gate="G$1" x="27.94" y="205.74"/>
 </instances>
 <busses>

Commit message: value corrected
Other:
- note added: "0R for SSR FDD2510"
Changed lines of the file:
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@@
 <text x="223.52" y="25.4" size="1.778" layer="94">Input 1 (Option)</text>
 <text x="261.62" y="25.4" size="1.778" layer="94">Indicator LED</text>
+<text x="35.56" y="182.88" size="1.778" layer="91">0R for SSR FDD2510</text>
+<text x="114.3" y="182.88" size="1.778" layer="91">0R for SSR FDD2510</text>
 </plain>
 <instances>
